File: PCBfiles/Welduino.brd (EAGLE design)
At the start: 99.9 x 75.4 mm, 26 parts, among them IC1 REG1117, U1 ESP8266_ESP-01

Commit message: update
Parts:
- added LCD1: LCD_2X16_SIL, lcd_2x16_led_backlight:HY-1602F
Connections:
- new net 10K_POTENTIOMETER: LCD1.3
- new net N$22: LCD1.7
- new net N$23: LCD1.8
- new net N$24: LCD1.9
- new net N$25: LCD1.10
- net 5V: now also LCD1.15, LCD1.2
- net GND: now also LCD1.1, LCD1.16, LCD1.5
- net LCD_2: now also LCD1.4
- net LCD_4: now also LCD1.6
- net LCD_5: now also LCD1.11
- net LCD_6: now also LCD1.12
- net LCD_7: now also LCD1.13
- net LCD_8: now also LCD1.14
Changed lines of the file:
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@@
 <attribute name="VALUE" x="1.22715" y="7.756234375" size="1.27" layer="27" ratio="10"/>
+</element>
+<element name="LCD1" library="lcd_2x16_led_backlight" package="HY-1602F" value="LCD_2X16_SIL" x="4.9028" y="-6.4788" smashed="yes">
+<attribute name="NAME" x="-0.5572" y="-3.6788" size="1.27" layer="25"/>
 </element>
 </elements>
@@
 <contactref element="X4" pad="1"/>
 <contactref element="X6" pad="1"/>
+<contactref element="LCD1" pad="2"/>
+<contactref element="LCD1" pad="15"/>
 <wire x1="18.6578875" y1="37.88495" x2="27.72918125" y2="70.631015625" width="0" layer="19" extent="1-1"/>
 <wire x1="18.7098625" y1="33.790884375" x2="18.6578875" y2="37.88495" width="0" layer="19" extent="1-1"/>
 <wire x1="7.231740625" y1="34.696978125" x2="18.7098625" y2="33.790884375" width="0" layer="19" extent="1-1"/>
+<wire x1="14.0636625" y1="14.107125" x2="18.7098625" y2="33.790884375" width="0" layer="19" extent="1-1"/>
+<wire x1="34.762528125" y1="14.107125" x2="14.0636625" y2="14.107125" width="0" layer="19" extent="1-1"/>
+<wire x1="55.38645" y1="14.157890625" x2="34.762528125" y2="14.107125" width="0" layer="19" extent="1-1"/>
 <wire x1="39.6311125" y1="38.13814375" x2="18.6578875" y2="37.88495" width="0" layer="19" extent="1-1"/>
 <wire x1="39.6311125" y1="36.53814375" x2="39.6311125" y2="38.13814375" width="0" layer="19" extent="1-1"/>
@@
 <wire x1="55.265625" y1="35.449490625" x2="52.238625" y2="35.39949375" width="0" layer="19" extent="1-1"/>
 <wire x1="57.914646875" y1="35.451415625" x2="55.265625" y2="35.449490625" width="0" layer="19" extent="1-1"/>
-<wire x1="55.38645" y1="14.157890625" x2="18.7098625" y2="33.790884375" width="0" layer="19" extent="1-1"/>
-<wire x1="34.762528125" y1="14.107125" x2="55.38645" y2="14.157890625" width="0" layer="19" extent="1-1"/>
-<wire x1="14.0636625" y1="14.107125" x2="34.762528125" y2="14.107125" width="0" layer="19" extent="1-1"/>
+<wire x1="9.9828" y1="-6.4788" x2="14.0636625" y2="14.107125" width="0" layer="19" extent="1-1"/>
+<wire x1="43.0028" y1="-6.4788" x2="34.762528125" y2="14.107125" width="0" layer="19" extent="1-1"/>
 </signal>
 <signal name="N$2">
@@
 <contactref element="X5" pad="1"/>
 <contactref element="X1" pad="1"/>
+<contactref element="LCD1" pad="5"/>
+<contactref element="LCD1" pad="16"/>
+<contactref element="LCD1" pad="1"/>
 <wire x1="31.730709375" y1="67.029403125" x2="35.49" y2="70.21" width="0" layer="19" extent="1-1"/>
 <wire x1="27.72918125" y1="66.059015625" x2="31.730709375" y2="67.029403125" width="0" layer="19" extent="1-1"/>
@@
 <wire x1="28.039315625" y1="30.92004375" x2="28.074215625" y2="34.337440625" width="0" layer="19" extent="1-1"/>
 <wire x1="25.0048" y1="30.9051375" x2="28.039315625" y2="30.92004375" width="0" layer="19" extent="1-1"/>
+<wire x1="24.376128125" y1="14.107125" x2="25.0048" y2="30.9051375" width="0" layer="19" extent="1-1"/>
 <wire x1="7.231740625" y1="29.696978125" x2="25.0048" y2="30.9051375" width="0" layer="19" extent="1-1"/>
-<wire x1="45.074490625" y1="14.157890625" x2="7.231740625" y2="29.696978125" width="0" layer="19" extent="1-1"/>
-<wire x1="24.376128125" y1="14.107125" x2="45.074490625" y2="14.157890625" width="0" layer="19" extent="1-1"/>
+<wire x1="45.074490625" y1="14.157890625" x2="24.376128125" y2="14.107125" width="0" layer="19" extent="1-1"/>
 <wire x1="65.700125" y1="14.1579125" x2="45.074490625" y2="14.157890625" width="0" layer="19" extent="1-1"/>
+<wire x1="45.5428" y1="-6.4788" x2="45.074490625" y2="14.157890625" width="0" layer="19" extent="1-1"/>
+<wire x1="17.6028" y1="-6.4788" x2="24.376128125" y2="14.107125" width="0" layer="19" extent="1-1"/>
+<wire x1="7.4428" y1="-6.4788" x2="17.6028" y2="-6.4788" width="0" layer="19" extent="1-1"/>
 </signal>
 <signal name="N$26">
@@
 <signal name="LCD_2">
 <contactref element="328-1" pad="32"/>
+<contactref element="LCD1" pad="4"/>
+<wire x1="15.0628" y1="-6.4788" x2="40.9967125" y2="42.15774375" width="0" layer="19" extent="1-1"/>
 </signal>
 <signal name="LCD_4">
 <contactref element="328-1" pad="2"/>
+<contactref element="LCD1" pad="6"/>
+<wire x1="20.1428" y1="-6.4788" x2="39.6311125" y2="39.73814375" width="0" layer="19" extent="1-1"/>
 </signal>
 <signal name="LCD_5">
 <contactref element="328-1" pad="9"/>
+<contactref element="LCD1" pad="11"/>
+<wire x1="32.8428" y1="-6.4788" x2="40.9967125" y2="33.31854375" width="0" layer="19" extent="1-1"/>
 </signal>
 <signal name="LCD_6">
 <contactref element="328-1" pad="10"/>
+<contactref element="LCD1" pad="12"/>
+<wire x1="35.3828" y1="-6.4788" x2="41.7967125" y2="33.57254375" width="0" layer="19" extent="1-1"/>
 </signal>
 <signal name="LCD_7">
 <contactref element="328-1" pad="11"/>
+<contactref element="LCD1" pad="13"/>
+<wire x1="37.9228" y1="-6.4788" x2="42.5967125" y2="33.57254375" width="0" layer="19" extent="1-1"/>
 </signal>
 <signal name="LCD_8">
 <contactref element="328-1" pad="12"/>
+<contactref element="LCD1" pad="14"/>
+<wire x1="40.4628" y1="-6.4788" x2="43.3967125" y2="33.57254375" width="0" layer="19" extent="1-1"/>
 </signal>
 <signal name="ENCODER_A3">
@@
 <contactref element="328-1" pad="13"/>
 </signal>
+<signal name="10K_POTENTIOMETER">
+<contactref element="LCD1" pad="3"/>
+</signal>
+<signal name="N$22">
+<contactref element="LCD1" pad="7"/>
+</signal>
+<signal name="N$23">
+<contactref element="LCD1" pad="8"/>
+</signal>
+<signal name="N$24">
+<contactref element="LCD1" pad="9"/>
+</signal>
+<signal name="N$25">
+<contactref element="LCD1" pad="10"/>
+</signal>
 </signals>

Commit message: update
Parts:
- added R3: (no value), pot:3223J
Connections:
- new net RELAY_PIN_CURRENT_ON_12: X5.2
- new net RELAY_PIN_GAS_ON_3: X6.2
- net 10K_POTENTIOMETER: now also R3.2
- net 5V: now also R3.1, X5.1
- net GND: now also R3.3; no longer X5.1
- net PIN_CURRENT_ON_12: no longer X5.2
- net PIN_GAS_ON_3: no longer X6.2
Other:
- board text removed: "grbl"
Changed lines of the file:
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@@
 <plain>
 <text x="1.809459375" y="28.707753125" size="1.55" layer="1" font="vector" rot="R90">POWER</text>
-<text x="80.567175" y="27.784740625" size="1.55" layer="1" font="vector">grbl</text>
 <wire x1="-1.04" y1="60.47" x2="-1.04" y2="-1.2" width="1" layer="46"/>
 <wire x1="-1.04" y1="-1.2" x2="98.9" y2="-1.2" width="1" layer="46"/>
@@
 <attribute name="NAME" x="-0.5572" y="-3.6788" size="1.27" layer="25"/>
 </element>
+<element name="R3" library="pot" library_urn="urn:adsk.eagle:library:331" package="3223J" package3d_urn="urn:adsk.eagle:package:22724/1" value="" x="5.8601625" y="5.346865625" smashed="yes">
+<attribute name="NAME" x="4.2726625" y="7.569365625" size="1.27" layer="25"/>
+<attribute name="POPULARITY" value="0" x="5.8601625" y="5.346865625" size="1.778" layer="27" display="off"/>
+<attribute name="VALUE" x="3.9551625" y="1.854365625" size="1.27" layer="27"/>
+</element>
 </elements>
 <signals>
@@
 <contactref element="LCD1" pad="2"/>
 <contactref element="LCD1" pad="15"/>
+<contactref element="R3" pad="1"/>
+<contactref element="X5" pad="1"/>
 <wire x1="18.6578875" y1="37.88495" x2="27.72918125" y2="70.631015625" width="0" layer="19" extent="1-1"/>
 <wire x1="18.7098625" y1="33.790884375" x2="18.6578875" y2="37.88495" width="0" layer="19" extent="1-1"/>
 <wire x1="7.231740625" y1="34.696978125" x2="18.7098625" y2="33.790884375" width="0" layer="19" extent="1-1"/>
 <wire x1="14.0636625" y1="14.107125" x2="18.7098625" y2="33.790884375" width="0" layer="19" extent="1-1"/>
-<wire x1="34.762528125" y1="14.107125" x2="14.0636625" y2="14.107125" width="0" layer="19" extent="1-1"/>
+<wire x1="24.376128125" y1="14.107125" x2="14.0636625" y2="14.107125" width="0" layer="19" extent="1-1"/>
+<wire x1="34.762528125" y1="14.107125" x2="24.376128125" y2="14.107125" width="0" layer="19" extent="1-1"/>
+<wire x1="3.8601625" y1="6.746865625" x2="14.0636625" y2="14.107125" width="0" layer="19" extent="1-1"/>
+<wire x1="9.9828" y1="-6.4788" x2="3.8601625" y2="6.746865625" width="0" layer="19" extent="1-1"/>
 <wire x1="55.38645" y1="14.157890625" x2="34.762528125" y2="14.107125" width="0" layer="19" extent="1-1"/>
 <wire x1="39.6311125" y1="38.13814375" x2="18.6578875" y2="37.88495" width="0" layer="19" extent="1-1"/>
@@
 <wire x1="55.265625" y1="35.449490625" x2="52.238625" y2="35.39949375" width="0" layer="19" extent="1-1"/>
 <wire x1="57.914646875" y1="35.451415625" x2="55.265625" y2="35.449490625" width="0" layer="19" extent="1-1"/>
-<wire x1="9.9828" y1="-6.4788" x2="14.0636625" y2="14.107125" width="0" layer="19" extent="1-1"/>
 <wire x1="43.0028" y1="-6.4788" x2="34.762528125" y2="14.107125" width="0" layer="19" extent="1-1"/>
 </signal>
@@
 <contactref element="IC1" pad="1"/>
 <contactref element="X3" pad="1"/>
-<contactref element="X5" pad="1"/>
 <contactref element="X1" pad="1"/>
 <contactref element="LCD1" pad="5"/>
 <contactref element="LCD1" pad="16"/>
 <contactref element="LCD1" pad="1"/>
+<contactref element="R3" pad="3"/>
 <wire x1="31.730709375" y1="67.029403125" x2="35.49" y2="70.21" width="0" layer="19" extent="1-1"/>
 <wire x1="27.72918125" y1="66.059015625" x2="31.730709375" y2="67.029403125" width="0" layer="19" extent="1-1"/>
@@
 <wire x1="28.039315625" y1="30.92004375" x2="28.074215625" y2="34.337440625" width="0" layer="19" extent="1-1"/>
 <wire x1="25.0048" y1="30.9051375" x2="28.039315625" y2="30.92004375" width="0" layer="19" extent="1-1"/>
-<wire x1="24.376128125" y1="14.107125" x2="25.0048" y2="30.9051375" width="0" layer="19" extent="1-1"/>
 <wire x1="7.231740625" y1="29.696978125" x2="25.0048" y2="30.9051375" width="0" layer="19" extent="1-1"/>
-<wire x1="45.074490625" y1="14.157890625" x2="24.376128125" y2="14.107125" width="0" layer="19" extent="1-1"/>
+<wire x1="45.074490625" y1="14.157890625" x2="39.6311125" y2="37.33814375" width="0" layer="19" extent="1-1"/>
 <wire x1="65.700125" y1="14.1579125" x2="45.074490625" y2="14.157890625" width="0" layer="19" extent="1-1"/>
 <wire x1="45.5428" y1="-6.4788" x2="45.074490625" y2="14.157890625" width="0" layer="19" extent="1-1"/>
-<wire x1="17.6028" y1="-6.4788" x2="24.376128125" y2="14.107125" width="0" layer="19" extent="1-1"/>
-<wire x1="7.4428" y1="-6.4788" x2="17.6028" y2="-6.4788" width="0" layer="19" extent="1-1"/>
+<wire x1="3.8601625" y1="3.946865625" x2="7.231740625" y2="29.696978125" width="0" layer="19" extent="1-1"/>
+<wire x1="7.4428" y1="-6.4788" x2="3.8601625" y2="3.946865625" width="0" layer="19" extent="1-1"/>
+<wire x1="17.6028" y1="-6.4788" x2="7.4428" y2="-6.4788" width="0" layer="19" extent="1-1"/>
 </signal>
 <signal name="N$26">
@@
 <signal name="PIN_GAS_ON_3">
 <contactref element="328-1" pad="1"/>
-<contactref element="X6" pad="2"/>
-<wire x1="19.0636625" y1="14.107125" x2="39.3771125" y2="40.53814375" width="0" layer="19" extent="1-1"/>
 </signal>
 <signal name="PIN_THERMAL_SAFETY_13">
@@
 <signal name="PIN_CURRENT_ON_12">
 <contactref element="328-1" pad="16"/>
-<contactref element="X5" pad="2"/>
-<wire x1="29.376128125" y1="14.107125" x2="46.5967125" y2="33.31854375" width="0" layer="19" extent="1-1"/>
 </signal>
 <signal name="PIN_CURRENT_READ_A2">
@@
 <signal name="10K_POTENTIOMETER">
 <contactref element="LCD1" pad="3"/>
+<contactref element="R3" pad="2"/>
+<wire x1="12.5228" y1="-6.4788" x2="7.8601625" y2="5.346865625" width="0" layer="19" extent="1-1"/>
 </signal>
 <signal name="N$22">
@@
 <contactref element="LCD1" pad="10"/>
 </signal>
+<signal name="RELAY_PIN_GAS_ON_3">
+<contactref element="X6" pad="2"/>
+</signal>
+<signal name="RELAY_PIN_CURRENT_ON_12">
+<contactref element="X5" pad="2"/>
+</signal>
 </signals>
