File: PCBfiles/Welduino.sch (EAGLE design)
At the start: 26 parts, among them IC1 REG1117, U1 ESP8266_ESP-01

Commit message: update
Parts:
- added LCD1: LCD_2X16_SIL, lcd_2x16_led_backlight:LCD_2X16_SIL
Connections:
- new net 10K_POTENTIOMETER: LCD1.VO
- new net N$22: LCD1.DB0
- new net N$23: LCD1.DB1
- new net N$24: LCD1.DB2
- new net N$25: LCD1.DB3
- net 5V: now also LCD1.LEDA, LCD1.VCC
- net GND: now also LCD1.LEDK, LCD1.R/W, LCD1.VSS
- net LCD_2: now also LCD1.RS
- net LCD_4: now also LCD1.E
- net LCD_5: now also LCD1.DB4
- net LCD_6: now also LCD1.DB5
- net LCD_7: now also LCD1.DB6
- net LCD_8: now also LCD1.DB7
Other:
- note added: "LCD"
Changed lines of the file:
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@@
 <part name="X6" library="con-wago-500" library_urn="urn:adsk.eagle:library:195" deviceset="W237-102" device="" package3d_urn="urn:adsk.eagle:package:10688/1"/>
 <part name="X7" library="con-wago-500" library_urn="urn:adsk.eagle:library:195" deviceset="W237-102" device="" package3d_urn="urn:adsk.eagle:package:10688/1"/>
+<part name="LCD1" library="lcd_2x16_led_backlight" deviceset="LCD_2X16_SIL" device=""/>
 </parts>
 <sheets>
@@
 <text x="-19.05" y="109.22" size="1.778" layer="91">ATMEGA328P-AU</text>
 <text x="158.75" y="57.15" size="1.778" layer="91">B7</text>
+<text x="-83.82" y="109.22" size="1.778" layer="91">LCD</text>
 </plain>
 <instances>
@@
 <attribute name="VALUE" x="190.5" y="55.753" size="1.778" layer="96" rot="R180"/>
 <attribute name="NAME" x="187.96" y="51.181" size="1.778" layer="95"/>
+</instance>
+<instance part="LCD1" gate="G$1" x="-43.18" y="82.55" smashed="yes">
+<attribute name="NAME" x="-50.8" y="39.37" size="1.27" layer="95"/>
 </instance>
 </instances>
@@
 <label x="162.56" y="16.51" size="1.778" layer="95"/>
 </segment>
+<segment>
+<pinref part="LCD1" gate="G$1" pin="VCC"/>
+<wire x1="-55.88" y1="80.01" x2="-66.04" y2="80.01" width="0.1524" layer="91"/>
+<label x="-67.31" y="80.01" size="1.778" layer="95"/>
+</segment>
+<segment>
+<pinref part="LCD1" gate="G$1" pin="LEDA"/>
+<wire x1="-55.88" y1="46.99" x2="-66.04" y2="46.99" width="0.1524" layer="91"/>
+<label x="-67.31" y="46.99" size="1.778" layer="95"/>
+</segment>
 </net>
 <net name="N$2" class="0">
@@
 <label x="162.56" y="87.63" size="1.778" layer="95"/>
 </segment>
+<segment>
+<pinref part="LCD1" gate="G$1" pin="R/W"/>
+<wire x1="-55.88" y1="72.39" x2="-66.04" y2="72.39" width="0.1524" layer="91"/>
+<label x="-67.31" y="72.39" size="1.778" layer="95"/>
+</segment>
+<segment>
+<pinref part="LCD1" gate="G$1" pin="LEDK"/>
+<wire x1="-55.88" y1="44.45" x2="-66.04" y2="44.45" width="0.1524" layer="91"/>
+<label x="-67.31" y="44.45" size="1.778" layer="95"/>
+</segment>
+<segment>
+<pinref part="LCD1" gate="G$1" pin="VSS"/>
+<wire x1="-55.88" y1="82.55" x2="-66.04" y2="82.55" width="0.1524" layer="91"/>
+<label x="-67.31" y="82.55" size="1.778" layer="95"/>
+</segment>
 </net>
 <net name="N$26" class="0">
@@
 <label x="87.63" y="50.8" size="1.778" layer="95"/>
 </segment>
+<segment>
+<pinref part="LCD1" gate="G$1" pin="RS"/>
+<wire x1="-55.88" y1="74.93" x2="-66.04" y2="74.93" width="0.1524" layer="91"/>
+<label x="-67.31" y="74.93" size="1.778" layer="95"/>
+</segment>
 </net>
 <net name="LCD_4" class="0">
@@
 <label x="87.63" y="43.18" size="1.778" layer="95"/>
 </segment>
+<segment>
+<pinref part="LCD1" gate="G$1" pin="E"/>
+<wire x1="-55.88" y1="69.85" x2="-66.04" y2="69.85" width="0.1524" layer="91"/>
+<label x="-67.31" y="69.85" size="1.778" layer="95"/>
+</segment>
 </net>
 <net name="LCD_5" class="0">
@@
 <label x="87.63" y="40.64" size="1.778" layer="95"/>
 </segment>
+<segment>
+<pinref part="LCD1" gate="G$1" pin="DB4"/>
+<wire x1="-55.88" y1="57.15" x2="-66.04" y2="57.15" width="0.1524" layer="91"/>
+<label x="-67.31" y="57.15" size="1.778" layer="95"/>
+</segment>
 </net>
 <net name="LCD_6" class="0">
@@
 <label x="87.63" y="38.1" size="1.778" layer="95"/>
 </segment>
+<segment>
+<pinref part="LCD1" gate="G$1" pin="DB5"/>
+<wire x1="-55.88" y1="54.61" x2="-66.04" y2="54.61" width="0.1524" layer="91"/>
+<label x="-67.31" y="54.61" size="1.778" layer="95"/>
+</segment>
 </net>
 <net name="LCD_7" class="0">
@@
 <label x="87.63" y="35.56" size="1.778" layer="95"/>
 </segment>
+<segment>
+<pinref part="LCD1" gate="G$1" pin="DB6"/>
+<wire x1="-55.88" y1="52.07" x2="-66.04" y2="52.07" width="0.1524" layer="91"/>
+<label x="-67.31" y="52.07" size="1.778" layer="95"/>
+</segment>
 </net>
 <net name="LCD_8" class="0">
@@
 <label x="87.63" y="33.02" size="1.778" layer="95"/>
 </segment>
+<segment>
+<pinref part="LCD1" gate="G$1" pin="DB7"/>
+<wire x1="-55.88" y1="49.53" x2="-66.04" y2="49.53" width="0.1524" layer="91"/>
+<label x="-67.31" y="49.53" size="1.778" layer="95"/>
+</segment>
 </net>
 <net name="ENCODER_A3" class="0">
@@
 </segment>
 </net>
+<net name="N$15" class="0">
+<segment>
+<wire x1="-29.21" y1="114.3" x2="-87.63" y2="114.3" width="0.1524" layer="91"/>
+<wire x1="-87.63" y1="114.3" x2="-87.63" y2="106.68" width="0.1524" layer="91"/>
+<wire x1="-87.63" y1="106.68" x2="-87.63" y2="10.16" width="0.1524" layer="91"/>
+<wire x1="-87.63" y1="10.16" x2="-29.21" y2="8.89" width="0.1524" layer="91"/>
+<wire x1="-29.21" y1="8.89" x2="-29.21" y2="106.68" width="0.1524" layer="91"/>
+<wire x1="-29.21" y1="114.3" x2="-29.21" y2="106.68" width="0.1524" layer="91"/>
+<wire x1="-29.21" y1="106.68" x2="-87.63" y2="106.68" width="0.1524" layer="91"/>
+</segment>
+</net>
+<net name="10K_POTENTIOMETER" class="0">
+<segment>
+<pinref part="LCD1" gate="G$1" pin="VO"/>
+<wire x1="-55.88" y1="77.47" x2="-66.04" y2="77.47" width="0.1524" layer="91"/>
+<label x="-83.82" y="77.47" size="1.778" layer="95"/>
+</segment>
+<segment>
+<wire x1="-76.2" y1="25.4" x2="-69.85" y2="25.4" width="0.1524" layer="91"/>
+<label x="-83.82" y="24.13" size="1.778" layer="95"/>
+</segment>
+</net>
+<net name="N$22" class="0">
+<segment>
+<pinref part="LCD1" gate="G$1" pin="DB0"/>
+<wire x1="-55.88" y1="67.31" x2="-66.04" y2="67.31" width="0.1524" layer="91"/>
+</segment>
+</net>
+<net name="N$23" class="0">
+<segment>
+<pinref part="LCD1" gate="G$1" pin="DB1"/>
+<wire x1="-55.88" y1="64.77" x2="-66.04" y2="64.77" width="0.1524" layer="91"/>
+</segment>
+</net>
+<net name="N$24" class="0">
+<segment>
+<pinref part="LCD1" gate="G$1" pin="DB2"/>
+<wire x1="-55.88" y1="62.23" x2="-66.04" y2="62.23" width="0.1524" layer="91"/>
+</segment>
+</net>
+<net name="N$25" class="0">
+<segment>
+<pinref part="LCD1" gate="G$1" pin="DB3"/>
+<wire x1="-55.88" y1="59.69" x2="-66.04" y2="59.69" width="0.1524" layer="91"/>
+</segment>
+</net>
+<net name="N$17" class="0">
+<segment>
+<wire x1="-63.5" y1="27.94" x2="-55.88" y2="27.94" width="0.1524" layer="91"/>
+</segment>
+</net>
+<net name="N$18" class="0">
+<segment>
+<wire x1="-63.5" y1="22.86" x2="-55.88" y2="22.86" width="0.1524" layer="91"/>
+</segment>
+</net>

Commit message: update
Parts:
- added R3: (no value), pot:TRIM_EU-3223J
Connections:
- new net RELAY_PIN_CURRENT_ON_12: X5-2.KL
- new net RELAY_PIN_GAS_ON_3: X6-2.KL
- net 10K_POTENTIOMETER: now also R3.S
- net 5V: now also R3.A, X5-1.KL
- net GND: now also R3.E; no longer X5-1.KL
- net PIN_CURRENT_ON_12: no longer X5-2.KL
- net PIN_GAS_ON_3: no longer X6-2.KL
Other:
- moved on the sheet: LCD1
